File: de0-nano-c64.kicad_sch (KiCad schematic)
At the start: 51 parts, among them J1 GPIO_0, J10 SD_Card, J2 PS2_0, J3 PS2_1, J4 AUDIO_L, J5 GPIO_1, J6 VGA_OUT, J7 AUDIO_R, J8 JOYSTICK_1, J9 JOYSTICK_2

Commit message: .
Parts:
- removed J4: AUDIO_L, 000_LOCAL:RCA, symbol 000_LOCAL:Conn_Coaxial
- removed J7: AUDIO_R, 000_LOCAL:RCA, symbol 000_LOCAL:Conn_Coaxial
- added J11: AudioJack3, Connector_Audio:Jack_3.5mm_CUI_SJ1-3523N_Horizontal, symbol Connector_Audio:AudioJack3
Connections:
- net GND: now also J11.S
- net at C1.1, R22.2: now also J11.T
- net at C2.1, R23.2: now also J11.R
Changed lines of the file:
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@@
+    (stroke (width 0) (type default))
+  )
+  (wire (pts (xy 172.72 41.91) (xy 176.53 41.91))
     (stroke (width 0) (type default))
   )
@@
     (stroke (width 0) (type default))
   )
+  (wire (pts (xy 172.72 29.21) (xy 172.72 39.37))
+    (stroke (width 0) (type default))
+  )
   (wire (pts (xy 162.56 29.21) (xy 165.1 29.21))
     (stroke (width 0) (type default))
@@
     (stroke (width 0) (type default))
   )
+  (wire (pts (xy 172.72 39.37) (xy 176.53 39.37))
+    (stroke (width 0) (type default))
+  )
   (wire (pts (xy 264.16 49.53) (xy 271.78 49.53))
     (stroke (width 0) (type default))
@@
   )
   (wire (pts (xy 158.75 91.44) (xy 171.45 91.44))
+    (stroke (width 0) (type default))
+  )
+  (wire (pts (xy 172.72 48.26) (xy 172.72 41.91))
     (stroke (width 0) (type default))
   )
@@
     )
   )
-  (symbol (lib_id "000_LOCAL:GND") (at 177.8 53.34 0) (unit 1)
+  (symbol (lib_id "000_LOCAL:GND") (at 176.53 44.45 0) (unit 1)
     (in_bom yes) (on_board yes) (dnp no) (fields_autoplaced)
-    (property "Reference" "#PWR06" (at 177.8 59.69 0)
-      (effects (font (size 1.27 1.27)) hide)
-    )
-    (property "Value" "GND" (at 177.8 58.42 0)
-      (effects (font (size 1.27 1.27)))
-    )
-    (property "Footprint" "" (at 177.8 53.34 0)
-      (effects (font (size 1.27 1.27)) hide)
-    )
-    (property "Datasheet" "" (at 177.8 53.34 0)
+    (property "Reference" "#PWR06" (at 176.53 50.8 0)
+      (effects (font (size 1.27 1.27)) hide)
+    )
+    (property "Value" "GND" (at 176.53 49.53 0)
+      (effects (font (size 1.27 1.27)))
+    )
+    (property "Footprint" "" (at 176.53 44.45 0)
+      (effects (font (size 1.27 1.27)) hide)
+    )
+    (property "Datasheet" "" (at 176.53 44.45 0)
       (effects (font (size 1.27 1.27)) hide)
     )
@@
         (path "/dc38b7f3-94d8-459d-903b-54a6ae2cb037"
           (reference "#PWR06") (unit 1)
+        )
+      )
+    )
+  )
+  (symbol (lib_id "Connector_Audio:AudioJack3") (at 181.61 41.91 180) (unit 1)
+    (in_bom yes) (on_board yes) (dnp no) (fields_autoplaced)
+    (property "Reference" "J11" (at 189.23 40.005 0)
+      (effects (font (size 1.27 1.27)) (justify right))
+    )
+    (property "Value" "AudioJack3" (at 189.23 42.545 0)
+      (effects (font (size 1.27 1.27)) (justify right))
+    )
+    (property "Footprint" "Connector_Audio:Jack_3.5mm_CUI_SJ1-3523N_Horizontal" (at 181.61 41.91 0)
+      (effects (font (size 1.27 1.27)) hide)
+    )
+    (property "Datasheet" "~" (at 181.61 41.91 0)
+      (effects (font (size 1.27 1.27)) hide)
+    )
+    (pin "T")
+    (pin "S")
+    (pin "R")
+    (instances
+      (project "de0-nano-c64"
+        (path "/dc38b7f3-94d8-459d-903b-54a6ae2cb037"
+          (reference "J11") (unit 1)
         )
       )
@@
         (path "/dc38b7f3-94d8-459d-903b-54a6ae2cb037"
           (reference "R15") (unit 1)
-        )
-      )
-    )
-  )
-  (symbol (lib_id "000_LOCAL:Conn_Coaxial") (at 177.8 48.26 0) (unit 1)
-    (in_bom yes) (on_board yes) (dnp no) (fields_autoplaced)
-    (property "Reference" "J7" (at 181.61 47.2832 0)
-      (effects (font (size 1.27 1.27)) (justify left))
-    )
-    (property "Value" "AUDIO_R" (at 181.61 49.8232 0)
-      (effects (font (size 1.27 1.27)) (justify left))
-    )
-    (property "Footprint" "000_LOCAL:RCA" (at 177.8 48.26 0)
-      (effects (font (size 1.27 1.27)) hide)
-    )
-    (property "Datasheet" " ~" (at 177.8 48.26 0)
-      (effects (font (size 1.27 1.27)) hide)
-    )
-    (pin "2")
-    (pin "1")
-    (instances
-      (project "de0-nano-c64"
-        (path "/dc38b7f3-94d8-459d-903b-54a6ae2cb037"
-          (reference "J7") (unit 1)
         )
       )
@@
         (path "/dc38b7f3-94d8-459d-903b-54a6ae2cb037"
           (reference "#FLG02") (unit 1)
-        )
-      )
-    )
-  )
-  (symbol (lib_id "000_LOCAL:Conn_Coaxial") (at 177.8 29.21 0) (unit 1)
-    (in_bom yes) (on_board yes) (dnp no) (fields_autoplaced)
-    (property "Reference" "J4" (at 181.61 28.2332 0)
-      (effects (font (size 1.27 1.27)) (justify left))
-    )
-    (property "Value" "AUDIO_L" (at 181.61 30.7732 0)
-      (effects (font (size 1.27 1.27)) (justify left))
-    )
-    (property "Footprint" "000_LOCAL:RCA" (at 177.8 29.21 0)
-      (effects (font (size 1.27 1.27)) hide)
-    )
-    (property "Datasheet" " ~" (at 177.8 29.21 0)
-      (effects (font (size 1.27 1.27)) hide)
-    )
-    (pin "2")
-    (pin "1")
-    (instances
-      (project "de0-nano-c64"
-        (path "/dc38b7f3-94d8-459d-903b-54a6ae2cb037"
-          (reference "J4") (unit 1)
         )
       )
@@
         )
       )
-    )
-  )
-  (symbol (lib_id "000_LOCAL:GND") (at 177.8 34.29 0) (unit 1)
-    (in_bom yes) (on_board yes) (dnp no) (fields_autoplaced)
-    (property "Reference" "#PWR04" (at 177.8 40.64 0)
-      (effects (font (size 1.27 1.27)) hide)
-    )
-    (property "Value" "GND" (at 177.8 39.37 0)
-      (effects (font (size 1.27 1.27)))
-    )
-    (property "Footprint" "" (at 177.8 34.29 0)
-      (effects (font (size 1.27 1.27)) hide)
-    )
-    (property "Datasheet" "" (at 177.8 34.29 0)
-      (effects (font (size 1.27 1.27)) hide)
-    )
-    (pin "1")
-    (instances
-      (project "de0-nano-c64"
-        (path "/dc38b7f3-94d8-459d-903b-54a6ae2cb037"
-          (reference "#PWR04") (unit 1)
-        )
-      )

Commit message: remove unusedfiles, update footprints and 3d models
Parts:
- J10: footprint Connector_Card:microSD_HC_Hirose_DM3AT-SF-PEJM5 -> 000_LOCAL:MOLEX_503398-1892; symbol Connector:Micro_SD_Card -> 000_LOCAL:Micro_SD_Card
- J11: value AudioJack3 -> AUDIO; footprint Connector_Audio:Jack_3.5mm_CUI_SJ1-3523N_Horizontal -> 000_LOCAL:Jack_3.5mm_CUI_SJ1-3523N_Horizontal; symbol Connector_Audio:AudioJack3 -> 000_LOCAL:AudioJack3
- J2, J3: symbol Connector:DIN-6 -> 000_LOCAL:Mini-DIN-6
- J6: value VGA_OUT -> VGA; footprint 000_LOCAL:HD15-SN-25 -> 000_LOCAL:AMPHENOL_ICD15S13E4GV00LF
- J8, J9: footprint Connector_Dsub:DSUB-9_Male_Horizontal_P2.77x2.84mm_EdgePinOffset4.94mm_Housed_MountingHolesOffset7.48mm -> Connector_Dsub:DSUB-9_Male_Horizontal_P2.77x2.84mm_EdgePinOffset7.70mm_Housed_MountingHolesOffset9.12mm; symbol Connector:DE9_Plug_MountingHoles -> 000_LOCAL:DE9_Plug_MountingHoles
Connections:
- net GND: now also J2.S1, J3.S1
Other:
- moved on the sheet: R17, R19

Commit message: start routing
Connections:
- net J1_DOWN: now also J5.7 (Pin_7); no longer J5.3 (Pin_3)
- net J1_FIRE: now also J5.1 (Pin_1); no longer J5.9 (Pin_9)
- net J1_RIGHT: now also J5.3 (Pin_3); no longer J5.7 (Pin_7)
- net J1_UP: now also J5.9 (Pin_9); no longer J5.1 (Pin_1)
- net J2_DOWN: now also J5.19 (Pin_19); no longer J5.15 (Pin_15)
- net J2_FIRE: now also J5.13 (Pin_13); no longer J5.21 (Pin_21)
- net J2_RIGHT: now also J5.15 (Pin_15); no longer J5.19 (Pin_19)
- net J2_UP: now also J5.21 (Pin_21); no longer J5.13 (Pin_13)
- net PS2_0_CLK: now also J5.36 (Pin_36); no longer J5.38 (Pin_38)
- net PS2_0_DAT: now also J5.34 (Pin_34); no longer J5.40 (Pin_40)
- net PS2_1_CLK: now also J5.40 (Pin_40); no longer J5.34 (Pin_34)
- net PS2_1_DAT: now also J5.38 (Pin_38); no longer J5.36 (Pin_36)
- net SD_CLK: now also J5.39 (Pin_39); no longer J5.37 (Pin_37)
- net SD_CMD: now also J5.33 (Pin_33); no longer J5.39 (Pin_39)
- net SD_DAT0: now also J5.31 (Pin_31); no longer J5.27 (Pin_27)
- net SD_DAT1: now also J5.27 (Pin_27); no longer J5.31 (Pin_31)
- net SD_DAT2: now also J5.37 (Pin_37); no longer J5.33 (Pin_33)
Changed lines of the file:
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@@
     (effects (font (size 1.27 1.27)) (justify left bottom))
   )
-  (label "J1_RIGHT" (at 93.98 39.37 180) (fields_autoplaced)
+  (label "J1_DOWN" (at 93.98 39.37 180) (fields_autoplaced)
     (effects (font (size 1.27 1.27)) (justify right bottom))
   )
@@
     (effects (font (size 1.27 1.27)) (justify left bottom))
   )
-  (label "J2_RIGHT" (at 93.98 54.61 180) (fields_autoplaced)
-    (effects (font (size 1.27 1.27)) (justify right bottom))
-  )
-  (label "PS2_0_CLK" (at 106.68 77.47 0) (fields_autoplaced)
-    (effects (font (size 1.27 1.27)) (justify left bottom))
-  )
-  (label "SD_CMD" (at 93.98 80.01 180) (fields_autoplaced)
+  (label "J2_DOWN" (at 93.98 54.61 180) (fields_autoplaced)
+    (effects (font (size 1.27 1.27)) (justify right bottom))
+  )
+  (label "PS2_1_DAT" (at 106.68 77.47 0) (fields_autoplaced)
+    (effects (font (size 1.27 1.27)) (justify left bottom))
+  )
+  (label "SD_CLK" (at 93.98 80.01 180) (fields_autoplaced)
     (effects (font (size 1.27 1.27)) (justify right bottom))
   )
@@
     (effects (font (size 1.27 1.27)) (justify right bottom))
   )
-  (label "J1_FIRE" (at 93.98 41.91 180) (fields_autoplaced)
+  (label "J1_UP" (at 93.98 41.91 180) (fields_autoplaced)
     (effects (font (size 1.27 1.27)) (justify right bottom))
   )
@@
     (effects (font (size 1.27 1.27)) (justify left bottom))
   )
-  (label "SD_DAT2" (at 93.98 72.39 180) (fields_autoplaced)
+  (label "SD_CMD" (at 93.98 72.39 180) (fields_autoplaced)
     (effects (font (size 1.27 1.27)) (justify right bottom))
   )
@@
     (effects (font (size 1.27 1.27)) (justify left bottom))
   )
-  (label "SD_DAT0" (at 93.98 64.77 180) (fields_autoplaced)
+  (label "SD_DAT1" (at 93.98 64.77 180) (fields_autoplaced)
     (effects (font (size 1.27 1.27)) (justify right bottom))
   )
@@
     (effects (font (size 1.27 1.27)) (justify left bottom))
   )
-  (label "PS2_1_DAT" (at 106.68 74.93 0) (fields_autoplaced)
+  (label "PS2_0_CLK" (at 106.68 74.93 0) (fields_autoplaced)
     (effects (font (size 1.27 1.27)) (justify left bottom))
   )
@@
     (effects (font (size 1.27 1.27)) (justify left bottom))
   )
-  (label "J2_FIRE" (at 93.98 57.15 180) (fields_autoplaced)
+  (label "J2_UP" (at 93.98 57.15 180) (fields_autoplaced)
     (effects (font (size 1.27 1.27)) (justify right bottom))
   )
@@
     (effects (font (size 1.27 1.27)) (justify left bottom))
   )
-  (label "J1_DOWN" (at 93.98 34.29 180) (fields_autoplaced)
+  (label "J1_RIGHT" (at 93.98 34.29 180) (fields_autoplaced)
     (effects (font (size 1.27 1.27)) (justify right bottom))
   )
@@
     (effects (font (size 1.27 1.27)) (justify left bottom))
   )
-  (label "SD_CLK" (at 93.98 77.47 180) (fields_autoplaced)
+  (label "SD_DAT2" (at 93.98 77.47 180) (fields_autoplaced)
     (effects (font (size 1.27 1.27)) (justify right bottom))
   )
@@
     (effects (font (size 1.27 1.27)) (justify left bottom))
   )
-  (label "J1_UP" (at 93.98 31.75 180) (fields_autoplaced)
-    (effects (font (size 1.27 1.27)) (justify right bottom))
-  )
-  (label "PS2_0_DAT" (at 106.68 80.01 0) (fields_autoplaced)
+  (label "J1_FIRE" (at 93.98 31.75 180) (fields_autoplaced)
+    (effects (font (size 1.27 1.27)) (justify right bottom))
+  )
+  (label "PS2_1_CLK" (at 106.68 80.01 0) (fields_autoplaced)
     (effects (font (size 1.27 1.27)) (justify left bottom))
   )
@@
     (effects (font (size 1.27 1.27)) (justify left bottom))
   )
-  (label "J2_UP" (at 93.98 46.99 180) (fields_autoplaced)
+  (label "J2_FIRE" (at 93.98 46.99 180) (fields_autoplaced)
     (effects (font (size 1.27 1.27)) (justify right bottom))
   )
@@
     (effects (font (size 1.27 1.27)) (justify right bottom))
   )
-  (label "J2_DOWN" (at 93.98 49.53 180) (fields_autoplaced)
-    (effects (font (size 1.27 1.27)) (justify right bottom))
-  )
-  (label "SD_DAT1" (at 93.98 69.85 180) (fields_autoplaced)
+  (label "J2_RIGHT" (at 93.98 49.53 180) (fields_autoplaced)
+    (effects (font (size 1.27 1.27)) (justify right bottom))
+  )
+  (label "SD_DAT0" (at 93.98 69.85 180) (fields_autoplaced)
     (effects (font (size 1.27 1.27)) (justify right bottom))
   )
@@
     (effects (font (size 1.27 1.27)) (justify left bottom))
   )
-  (label "PS2_1_CLK" (at 106.68 72.39 0) (fields_autoplaced)
-    (effects (font (size 1.27 1.27)) (justify left bottom))
-  )
+  (label "PS2_0_DAT" (at 106.68 72.39 0) (fields_autoplaced)
+    (effects (font (size 1.27 1.27)) (justify left bottom))
+  )

Commit message: finished traces
Connections:
- net J1_DOWN: now also J5.13 (Pin_13); no longer J5.7 (Pin_7)
- net J1_FIRE: now also J5.5 (Pin_5); no longer J5.1 (Pin_1)
- net J1_LEFT: now also J5.9 (Pin_9); no longer J5.5 (Pin_5)
- net J1_RIGHT: now also J5.7 (Pin_7); no longer J5.3 (Pin_3)
- net J1_UP: now also J5.15 (Pin_15); no longer J5.9 (Pin_9)
- net J2_DOWN: now also J5.23 (Pin_23); no longer J5.19 (Pin_19)
- net J2_FIRE: now also J5.17 (Pin_17); no longer J5.13 (Pin_13)
- net J2_LEFT: now also J5.21 (Pin_21); no longer J5.17 (Pin_17)
- net J2_RIGHT: now also J5.19 (Pin_19); no longer J5.15 (Pin_15)
- net J2_UP: now also J5.25 (Pin_25); no longer J5.21 (Pin_21)
- net PWM_L: now also J5.1 (Pin_1); no longer J5.23 (Pin_23)
- net PWM_R: now also J5.3 (Pin_3); no longer J5.25 (Pin_25)
Changed lines of the file:
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@@
     (effects (font (size 1.27 1.27)) (justify left bottom))
   )
-  (label "J1_DOWN" (at 93.98 39.37 180) (fields_autoplaced)
+  (label "J1_RIGHT" (at 93.98 39.37 180) (fields_autoplaced)
     (effects (font (size 1.27 1.27)) (justify right bottom))
   )
@@
     (effects (font (size 1.27 1.27)) (justify left bottom))
   )
-  (label "J2_DOWN" (at 93.98 54.61 180) (fields_autoplaced)
+  (label "J2_RIGHT" (at 93.98 54.61 180) (fields_autoplaced)
     (effects (font (size 1.27 1.27)) (justify right bottom))
   )
@@
     (effects (font (size 1.27 1.27)) (justify right bottom))
   )
-  (label "J1_UP" (at 93.98 41.91 180) (fields_autoplaced)
-    (effects (font (size 1.27 1.27)) (justify right bottom))
-  )
-  (label "PWM_L" (at 93.98 59.69 180) (fields_autoplaced)
+  (label "J1_LEFT" (at 93.98 41.91 180) (fields_autoplaced)
+    (effects (font (size 1.27 1.27)) (justify right bottom))
+  )
+  (label "J2_DOWN" (at 93.98 59.69 180) (fields_autoplaced)
     (effects (font (size 1.27 1.27)) (justify right bottom))
   )
@@
     (effects (font (size 1.27 1.27)) (justify right bottom))
   )
-  (label "J1_LEFT" (at 93.98 36.83 180) (fields_autoplaced)
+  (label "J1_FIRE" (at 93.98 36.83 180) (fields_autoplaced)
     (effects (font (size 1.27 1.27)) (justify right bottom))
   )
@@
     (effects (font (size 1.27 1.27)) (justify left bottom))
   )
-  (label "J2_UP" (at 93.98 57.15 180) (fields_autoplaced)
+  (label "J2_LEFT" (at 93.98 57.15 180) (fields_autoplaced)
     (effects (font (size 1.27 1.27)) (justify right bottom))
   )
@@
     (effects (font (size 1.27 1.27)) (justify left bottom))
   )
-  (label "J1_RIGHT" (at 93.98 34.29 180) (fields_autoplaced)
+  (label "PWM_R" (at 93.98 34.29 180) (fields_autoplaced)
     (effects (font (size 1.27 1.27)) (justify right bottom))
   )
@@
     (effects (font (size 1.27 1.27)) (justify left bottom))
   )
-  (label "J1_FIRE" (at 93.98 31.75 180) (fields_autoplaced)
+  (label "PWM_L" (at 93.98 31.75 180) (fields_autoplaced)
     (effects (font (size 1.27 1.27)) (justify right bottom))
   )
@@
     (effects (font (size 1.27 1.27)) (justify left bottom))
   )
-  (label "J2_FIRE" (at 93.98 46.99 180) (fields_autoplaced)
-    (effects (font (size 1.27 1.27)) (justify right bottom))
-  )
-  (label "PWM_R" (at 93.98 62.23 180) (fields_autoplaced)
-    (effects (font (size 1.27 1.27)) (justify right bottom))
-  )
-  (label "J2_RIGHT" (at 93.98 49.53 180) (fields_autoplaced)
+  (label "J1_DOWN" (at 93.98 46.99 180) (fields_autoplaced)
+    (effects (font (size 1.27 1.27)) (justify right bottom))
+  )
+  (label "J2_UP" (at 93.98 62.23 180) (fields_autoplaced)
+    (effects (font (size 1.27 1.27)) (justify right bottom))
+  )
+  (label "J1_UP" (at 93.98 49.53 180) (fields_autoplaced)
     (effects (font (size 1.27 1.27)) (justify right bottom))
   )
@@
     (effects (font (size 1.27 1.27)) (justify left bottom))
   )
-  (label "J2_LEFT" (at 93.98 52.07 180) (fields_autoplaced)
-    (effects (font (size 1.27 1.27)) (justify right bottom))
-  )
+  (label "J2_FIRE" (at 93.98 52.07 180) (fields_autoplaced)
+    (effects (font (size 1.27 1.27)) (justify right bottom))
+  )
