File: de0-nano-c64.kicad_pcb (KiCad board)
At the start: 2 copper layers, 71.6 x 84 mm, 52 parts, among them J1 GPIO_0, J10 SD_Card, J2 PS2_0, J3 PS2_1, J4 AUDIO_L, J5 GPIO_1, J6 VGA_OUT, J7 AUDIO_R, J8 JOYSTICK_1, J9 JOYSTICK_2

Commit message: .
Parts:
- removed J4: AUDIO_L, 000_LOCAL:RCA
- removed J7: AUDIO_R, 000_LOCAL:RCA
- added J11: AudioJack3, Connector_Audio:Jack_3.5mm_CUI_SJ1-3523N_Horizontal, F.Cu at (132.1, 70.6)
- moved J3 76.4 mm to (176.1, 130.9), turned to -90 degrees
- moved J2 71.5 mm to (176.1, 116.1), turned to -90 degrees
- moved C1 58.0 mm to (149.1, 72.6)
- moved R22 58.0 mm to (147.1, 72.6)
- moved C2 49.8 mm to (148.0, 67.8)
- moved R23 49.8 mm to (146.0, 67.8)
- moved R16 5.92 mm to (140.2, 72.9)
- moved R15 5.16 mm to (143.5, 70.5)
- moved R17 4.92 mm to (143.5, 74.2)
- moved R14 4.48 mm to (140.5, 68.5)
- moved J6 2.88 mm to (175.9, 91.3)
Routing:
- net GND: track 290.6 -> 150.1 mm
- net +5V: track 148.6 -> 39.3 mm
- net /PS2_0_DAT: track 68.4 -> 0.00 mm
- net /PS2_0_CLK: track 64.8 -> 0.00 mm
- net /PS2_1_DAT: track 57.0 -> 0.00 mm
- net /PS2_1_CLK: track 54.7 -> 0.00 mm
- net /J1_UP: track 67.8 -> 24.5 mm
- net +3V3: track 127.6 -> 85.0 mm, vias 4 -> 1
- net /PWM_L: track 26.3 -> 0.00 mm, vias 1 -> 0
- net /PWM_R: track 11.6 -> 0.00 mm
- net Net-(J2-Pad1): track 10.1 -> 0.00 mm
- net Net-(C1-Pad1): track 9.64 -> 0.07 mm
- net Net-(C2-Pad1): track 9.43 -> 0.07 mm
- net Net-(J3-Pad1): track 9.60 -> 0.28 mm
- net Net-(J2-Pad5): track 7.46 -> 0.00 mm
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Other:
- board size 71.6 x 84 mm -> 74.4 x 75.3 mm

Commit message: remove unusedfiles, update footprints and 3d models
Parts:
- J10: footprint Connector_Card:microSD_HC_Hirose_DM3AT-SF-PEJM5 -> 000_LOCAL:MOLEX_503398-1892
- J11: value AudioJack3 -> AUDIO; footprint Connector_Audio:Jack_3.5mm_CUI_SJ1-3523N_Horizontal -> 000_LOCAL:Jack_3.5mm_CUI_SJ1-3523N_Horizontal; moved to B.Cu
- J6: value VGA_OUT -> VGA; footprint 000_LOCAL:HD15-SN-25 -> 000_LOCAL:AMPHENOL_ICD15S13E4GV00LF
- J8, J9: footprint Connector_Dsub:DSUB-9_Male_Horizontal_P2.77x2.84mm_EdgePinOffset4.94mm_Housed_MountingHolesOffset7.48mm -> Connector_Dsub:DSUB-9_Male_Horizontal_P2.77x2.84mm_EdgePinOffset7.70mm_Housed_MountingHolesOffset9.12mm
- moved J11 22.3 mm to (154.4, 70.6), turned to 0 degrees
- moved R19 21.7 mm to (135.3, 69.7)
- moved R21 21.7 mm to (133.7, 69.7)
- moved R10 21.7 mm to (135.9, 75.5)
- moved R18 21.7 mm to (130.5, 69.7)
- moved R20 21.7 mm to (132.1, 69.7)
- moved R9 21.7 mm to (135.9, 73.5)
- moved C1 21.5 mm to (127.6, 71.2)
- moved C2 19.5 mm to (129.8, 75.0)
- moved J2 3.70 mm to (179.8, 116.0)
- moved J3 3.70 mm to (179.8, 130.9)
- moved J6 2.84 mm to (173.1, 91.3)
- moved J9 1.60 mm to (116.0, 128.4)
- moved J8 1.54 mm to (116.0, 96.3)
- moved J10 1.47 mm to (145.8, 133.8), turned to 180 degrees
Connections:
- J2 pad S1: (no net) -> GND
- J3 pad S1: (no net) -> GND
Routing:
- net GND: track 150.1 -> 0.00 mm
- net /VGA_H: track 41.8 -> 0.00 mm
- net +5V: track 39.3 -> 0.00 mm
- net /VGA_V: track 35.3 -> 0.00 mm
- net /SD_DAT1: track 29.1 -> 0.00 mm, vias 2 -> 0
- net /SD_CLK: track 25.6 -> 0.00 mm
- net /VGA_R: track 27.9 -> 5.40 mm
- net /SD_DAT3: track 22.4 -> 0.00 mm
- net /SD_CMD: track 22.0 -> 0.00 mm
- net /VGA_B: track 25.2 -> 5.40 mm
- net /VGA_G: track 24.2 -> 5.40 mm
- net /J1_FIRE: track 57.5 -> 39.7 mm
- net /J2_FIRE: track 65.4 -> 48.7 mm
- net /J2_DOWN: track 69.5 -> 54.7 mm
- net /J2_LEFT: track 64.4 -> 49.9 mm
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Other:
- board size 74.4 x 75.3 mm -> 79.4 x 75.3 mm

Commit message: start routing
Parts:
- R35, R36, R37, R38, R39: moved to B.Cu
- moved R19 70.9 mm to (170.1, 131.5), turned to 0 degrees
- moved R21 70.3 mm to (170.1, 129.9), turned to 180 degrees
- moved R20 69.8 mm to (170.1, 128.3), turned to 180 degrees
- moved R18 69.4 mm to (170.1, 126.7), turned to 0 degrees
- moved R14 53.1 mm to (170.1, 112.6), turned to 180 degrees
- moved R15 52.1 mm to (170.1, 115.3), turned to 180 degrees
- moved R13 50.6 mm to (180.3, 67.7)
- moved R17 50.5 mm to (170.1, 117.1), turned to 0 degrees
- moved R16 48.3 mm to (170.1, 110.8), turned to 0 degrees
- moved R1 47.4 mm to (180.3, 69.5)
- moved R2 44.3 mm to (180.3, 71.3)
- moved R31 41.8 mm to (157.2, 95.8), turned to 0 degrees
- moved R3 41.2 mm to (180.3, 73.1)
- moved R34 35.7 mm to (157.1, 98.5), turned to 0 degrees
- moved R33 34.9 mm to (157.0, 101.7), turned to 0 degrees
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Connections:
- J5 pad 1: /J1_UP -> /J1_FIRE
- J5 pad 13: /J2_UP -> /J2_FIRE
- J5 pad 15: /J2_DOWN -> /J2_RIGHT
- J5 pad 19: /J2_RIGHT -> /J2_DOWN
- J5 pad 21: /J2_FIRE -> /J2_UP
- J5 pad 27: /SD_DAT0 -> /SD_DAT1
- J5 pad 3: /J1_DOWN -> /J1_RIGHT
- J5 pad 31: /SD_DAT1 -> /SD_DAT0
- J5 pad 33: /SD_DAT2 -> /SD_CMD
- J5 pad 34: /PS2_1_CLK -> /PS2_0_DAT
- J5 pad 36: /PS2_1_DAT -> /PS2_0_CLK
- J5 pad 37: /SD_CLK -> /SD_DAT2
- J5 pad 38: /PS2_0_CLK -> /PS2_1_DAT
- J5 pad 39: /SD_CMD -> /SD_CLK
- J5 pad 40: /PS2_0_DAT -> /PS2_1_CLK
- J5 pad 7: /J1_RIGHT -> /J1_DOWN
- J5 pad 9: /J1_FIRE -> /J1_UP
Routing:
- net GND: track 0.00 -> 162.4 mm
- net +5V: track 0.00 -> 129.7 mm, vias 0 -> 1
- net /R3: track 8.85 -> 56.2 mm
- net /SD_DAT1: track 0.00 -> 44.3 mm, vias 0 -> 1
- net /R2: track 8.41 -> 50.5 mm
- net /J1_UP: track 11.8 -> 52.3 mm, vias 1 -> 0
- net /VGA_H: track 0.00 -> 40.0 mm, vias 0 -> 1
- net /R1: track 8.72 -> 47.0 mm
- net /SD_CMD: track 0.00 -> 35.4 mm, vias 0 -> 1
- net /SD_DAT3: track 0.00 -> 32.2 mm, vias 0 -> 1
- net /VGA_V: track 0.00 -> 31.7 mm, vias 0 -> 1
- net /R0: track 9.02 -> 38.9 mm
- net /VGA_R: track 5.40 -> 33.3 mm
- net /SD_CLK: track 0.00 -> 27.5 mm, vias 0 -> 1
- net /G3: track 8.86 -> 33.4 mm, vias 0 -> 1
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
Commit message: finished traces
Parts:
- moved C1 16.0 mm to (143.6, 71.7)
- moved C2 13.8 mm to (143.6, 75.9), turned to -90 degrees
- moved R23 8.10 mm to (145.8, 75.9), turned to 90 degrees
- moved R22 1.55 mm to (145.8, 71.7)
- moved R38 0.60 mm to (143.1, 123.5)
- moved J11 0.20 mm to (154.4, 70.4)
Connections:
- J5 pad 1: /J1_FIRE -> /PWM_L
- J5 pad 13: /J2_FIRE -> /J1_DOWN
- J5 pad 15: /J2_RIGHT -> /J1_UP
- J5 pad 17: /J2_LEFT -> /J2_FIRE
- J5 pad 19: /J2_DOWN -> /J2_RIGHT
- J5 pad 21: /J2_UP -> /J2_LEFT
- J5 pad 23: /PWM_L -> /J2_DOWN
- J5 pad 25: /PWM_R -> /J2_UP
- J5 pad 3: /J1_RIGHT -> /PWM_R
- J5 pad 5: /J1_LEFT -> /J1_FIRE
- J5 pad 7: /J1_DOWN -> /J1_RIGHT
- J5 pad 9: /J1_UP -> /J1_LEFT
Routing:
- net GND: track 162.4 -> 333.7 mm, vias 0 -> 2
- net +5V: track 129.7 -> 216.7 mm
- net +3V3: track 95.7 -> 142.9 mm, vias 13 -> 18
- net /PWM_L: track 0.00 -> 20.3 mm
- net /PWM_R: track 0.00 -> 18.9 mm
- net /J1_UP: track 52.3 -> 70.8 mm
- net Net-(C1-Pad1): track 0.07 -> 18.0 mm
- net /J1_DOWN: track 51.3 -> 67.9 mm
- net /SD_DAT0: track 26.8 -> 41.0 mm
- net /J1_LEFT: track 51.2 -> 64.0 mm
- net /J1_RIGHT: track 51.1 -> 60.3 mm
- net /J2_FIRE: track 69.8 -> 78.1 mm
- net Net-(J2-Pad1): track 2.17 -> 8.82 mm
- net Net-(C2-Pad1): track 0.07 -> 5.96 mm
- net /J1_FIRE: track 61.2 -> 66.2 mm
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Other:
- outline, holes or cut-outs redrawn

Commit message: finish
Parts:
- moved R20 0.94 mm to (170.1, 127.4)
- moved R18 0.87 mm to (170.1, 125.9)
- moved R17 0.86 mm to (170.1, 116.2)
- moved R39 0.65 mm to (140.1, 123.5)
- moved R19 0.59 mm to (170.1, 130.9)
- moved R15 0.58 mm to (170.1, 114.7)
- moved R21 0.51 mm to (170.1, 129.4)
- moved J10 0.44 mm to (145.8, 133.3)
- moved R14 0.33 mm to (170.1, 112.2)
Routing:
- net /J2_FIRE: track 78.1 -> 80.5 mm
- net /J2_RIGHT: track 62.3 -> 63.8 mm
- net GND: track 333.7 -> 335.1 mm
- net /PS2_1_DAT: track 5.45 -> 4.59 mm
- net /SD_CLK: track 27.5 -> 28.3 mm
- net /PS2_0_CLK: track 4.32 -> 5.09 mm
- net Net-(J3-Pad5): track 5.41 -> 5.92 mm
- added copper zone on B.Cu, net GND
- added copper zone on F.Cu, net GND
Other:
- outline, holes or cut-outs redrawn
- board text added: "DE0-Nano Commodore 64"
- board text added: "KEY0"
- board text added: "KEY1"
- board text added: "LED0"
- board text added: "LED1"
- board text added: "LED2"
- board text added: "LED3"
- board text added: "LED4"
- board text added: "LED5"
- board text added: "LED6"
- board text added: "LED7"
- board text removed: "<-USB"
- board text removed: "DAC TRIM"

Commit message: .
Other:
- board text added: "v1.0"
Changed lines of the file:
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@@
     (effects (font (size 1 1) (thickness 0.15) bold) (justify left bottom))
+  )
+  (gr_text "v1.0" (at 124.1425 71.755) (layer "F.SilkS")
+    (effects (font (size 2 2) (thickness 0.15)) (justify left))
   )
   (gr_text "DE0-Nano Commodore 64" (at 107.1245 68.199) (layer "F.SilkS")
